File: BTKeyboardAttempt.kicad_pcb (KiCad board)
At the start: 2 copper layers, 137 parts, among them J1 USB_C_Receptacle, SW1 SW_Push, U2 ATmega32U4-A, Y1 Crystal_GND24_Small

Commit message: Switch and Diode Routing
Parts:
- D1, D10, D11, D12, D13, D14, D15, D16, D17, D18, D19, D2, D20, D21, D22, D23, D24, D25, D26, D27, D28, D29, D3, D30, D31, D32, D33, D34, D35, D36, D37, D38, D39, D4, D40, D41, D42, D43, D44, D45, D46, D47, D48, D49, D5, D50, D51, D52, D53, D54, D55, D56, D57, D58, D59, D6, D60, D7, D8, D9, J1: moved to B.Cu
- SW1: footprint Diode_SMD:D_SOD-123 -> random-keyboard-parts:SKQG-1155865; moved to B.Cu
- moved Y1 316.4 mm to (365.1, 15.9)
- moved C7 300.7 mm to (366.7, 61.1)
- moved C6 299.0 mm to (361.9, 61.1)
- moved R6 298.5 mm to (361.2, 51.6)
- moved C5 297.2 mm to (357.2, 61.1)
- moved R5 296.6 mm to (356.4, 51.6)
- moved C4 295.5 mm to (352.4, 61.1)
- moved R4 294.8 mm to (351.6, 51.6)
- moved C3 293.7 mm to (347.7, 61.1)
- moved R3 293.0 mm to (346.9, 51.6)
- moved C2 292.0 mm to (342.9, 61.1)
- moved R2 291.2 mm to (342.1, 51.6)
- moved C1 290.2 mm to (338.1, 61.1)
- moved R1 289.4 mm to (337.3, 51.6)
- moved SW1 274.2 mm to (311.9, 34.1)
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Connections:
- MX1 pad 2: Net-(D2-A) -> Net-(D1-A)
- MX2 pad 2: Net-(D1-A) -> Net-(D2-A)
Routing:
- net ROW4: track 0.00 -> 209.6 mm
- net ROW2: track 0.00 -> 209.6 mm
- net ROW0: track 0.00 -> 209.6 mm
- net ROW3: track 0.00 -> 209.5 mm
- net ROW1: track 0.00 -> 209.5 mm
- net Net-(MX56-Pad1): track 0.00 -> 76.2 mm
- net Net-(MX51-Pad1): track 0.00 -> 76.2 mm
- net Net-(MX46-Pad1): track 0.00 -> 76.2 mm
- net Net-(MX41-Pad1): track 0.00 -> 76.2 mm
- net Net-(MX36-Pad1): track 0.00 -> 76.2 mm
- net Net-(MX31-Pad1): track 0.00 -> 76.2 mm
- net Net-(MX26-Pad1): track 0.00 -> 76.2 mm
- net Net-(MX21-Pad1): track 0.00 -> 76.2 mm
- net Net-(MX16-Pad1): track 0.00 -> 76.2 mm
- net Net-(MX11-Pad1): track 0.00 -> 76.2 mm
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
Commit message: Finished?
Parts:
- J1: footprint Connector_USB:USB_C_Receptacle_GCT_USB4125-xx-x_6P_TopMnt_Horizontal -> Connector_USB:USB_C_Receptacle_Amphenol_12401548E4-2A; moved to F.Cu
- U2: moved to F.Cu
- moved C7 250.1 mm to (118.4, 31.2), turned to 180 degrees
- moved Y1 247.4 mm to (118.4, 34.5)
- moved C6 244.7 mm to (118.4, 37.7), turned to 0 degrees
- moved C4 232.9 mm to (122.2, 26.5), turned to 180 degrees
- moved R4 231.2 mm to (122.2, 23.2), turned to 0 degrees
- moved C5 224.9 mm to (135.2, 25.5), turned to 0 degrees
- moved C3 222.4 mm to (125.9, 43.7), turned to 180 degrees
- moved C1 215.6 mm to (125.8, 24.2)
- moved C2 205.0 mm to (139.2, 38.7)
- moved R6 204.8 mm to (159.2, 17.2), turned to -90 degrees
- moved R1 201.0 mm to (136.5, 44.5), turned to 0 degrees
- moved R3 199.8 mm to (148.9, 24.9), turned to -90 degrees
- moved R5 199.5 mm to (159.2, 21.0)
- moved R2 191.3 mm to (152.6, 25.0), turned to -90 degrees
- moved U2 191.1 mm to (130.2, 34.7), turned to -90 degrees
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Connections:
- MX1 pad 1: Net-(MX1-Pad1) -> COL0
- MX10 pad 1: Net-(MX10-Pad1) -> COL1
- MX11 pad 1: Net-(MX11-Pad1) -> COL2
- MX12 pad 1: Net-(MX11-Pad1) -> COL2
- MX13 pad 1: Net-(MX11-Pad1) -> COL2
- MX14 pad 1: Net-(MX11-Pad1) -> COL2
- MX15 pad 1: Net-(MX11-Pad1) -> COL2
- MX16 pad 1: Net-(MX16-Pad1) -> COL3
- MX17 pad 1: Net-(MX16-Pad1) -> COL3
- MX18 pad 1: Net-(MX16-Pad1) -> COL3
- MX19 pad 1: Net-(MX16-Pad1) -> COL3
- MX2 pad 1: Net-(MX10-Pad1) -> COL1
- MX20 pad 1: Net-(MX16-Pad1) -> COL3
- MX21 pad 1: Net-(MX21-Pad1) -> COL4
- MX22 pad 1: Net-(MX21-Pad1) -> COL4
- MX23 pad 1: Net-(MX21-Pad1) -> COL4
- MX24 pad 1: Net-(MX21-Pad1) -> COL4
- MX25 pad 1: Net-(MX21-Pad1) -> COL4
- MX26 pad 1: Net-(MX26-Pad1) -> COL5
- MX27 pad 1: Net-(MX26-Pad1) -> COL5
- MX28 pad 1: Net-(MX26-Pad1) -> COL5
- MX29 pad 1: Net-(MX26-Pad1) -> COL5
- MX3 pad 1: Net-(MX1-Pad1) -> COL0
- MX30 pad 1: Net-(MX26-Pad1) -> COL5
- MX31 pad 1: Net-(MX31-Pad1) -> COL6
- MX32 pad 1: Net-(MX31-Pad1) -> COL6
- MX33 pad 1: Net-(MX31-Pad1) -> COL6
- MX34 pad 1: Net-(MX31-Pad1) -> COL6
- MX35 pad 1: Net-(MX31-Pad1) -> COL6
- MX36 pad 1: Net-(MX36-Pad1) -> COL7
- MX37 pad 1: Net-(MX36-Pad1) -> COL7
- MX38 pad 1: Net-(MX36-Pad1) -> COL7
- MX39 pad 1: Net-(MX36-Pad1) -> COL7
- MX4 pad 1: Net-(MX10-Pad1) -> COL1
- MX40 pad 1: Net-(MX36-Pad1) -> COL7
- MX41 pad 1: Net-(MX41-Pad1) -> COL8
- MX42 pad 1: Net-(MX41-Pad1) -> COL8
- MX43 pad 1: Net-(MX41-Pad1) -> COL8
- MX44 pad 1: Net-(MX41-Pad1) -> COL8
- MX45 pad 1: Net-(MX41-Pad1) -> COL8
- MX46 pad 1: Net-(MX46-Pad1) -> COL9
- MX47 pad 1: Net-(MX46-Pad1) -> COL9
- MX48 pad 1: Net-(MX46-Pad1) -> COL9
- MX49 pad 1: Net-(MX46-Pad1) -> COL9
- MX5 pad 1: Net-(MX1-Pad1) -> COL0
- MX50 pad 1: Net-(MX46-Pad1) -> COL9
- MX51 pad 1: Net-(MX51-Pad1) -> COL10
- MX52 pad 1: Net-(MX51-Pad1) -> COL10
- MX53 pad 1: Net-(MX51-Pad1) -> COL10
- MX54 pad 1: Net-(MX51-Pad1) -> COL10
- MX55 pad 1: Net-(MX51-Pad1) -> COL10
- MX56 pad 1: Net-(MX56-Pad1) -> COL11
- MX57 pad 1: Net-(MX56-Pad1) -> COL11
- MX58 pad 1: Net-(MX56-Pad1) -> COL11
- MX59 pad 1: Net-(MX56-Pad1) -> COL11
- MX6 pad 1: Net-(MX10-Pad1) -> COL1
- MX60 pad 1: Net-(MX56-Pad1) -> COL11
- MX7 pad 1: Net-(MX1-Pad1) -> COL0
- MX8 pad 1: Net-(MX10-Pad1) -> COL1
- MX9 pad 1: Net-(MX1-Pad1) -> COL0
- U2 pad 19: unconnected-(U2-PD1-Pad19) -> COL0
- U2 pad 20: unconnected-(U2-PD2-Pad20) -> COL1
- U2 pad 21: unconnected-(U2-PD3-Pad21) -> COL2
- U2 pad 22: unconnected-(U2-PD5-Pad22) -> COL3
- U2 pad 25: unconnected-(U2-PD4-Pad25) -> COL4
- U2 pad 26: unconnected-(U2-PD6-Pad26) -> COL5
- U2 pad 27: unconnected-(U2-PD7-Pad27) -> COL6
- U2 pad 28: unconnected-(U2-PB4-Pad28) -> COL7
- U2 pad 29: unconnected-(U2-PB5-Pad29) -> COL8
- U2 pad 30: unconnected-(U2-PB6-Pad30) -> COL9
- U2 pad 31: unconnected-(U2-PC6-Pad31) -> COL10
- U2 pad 32: unconnected-(U2-PC7-Pad32) -> COL11
- U2 pad 37: unconnected-(U2-PF6-Pad37) -> ROW0
- U2 pad 38: unconnected-(U2-PF5-Pad38) -> ROW1
- U2 pad 39: unconnected-(U2-PF4-Pad39) -> ROW2
- U2 pad 40: unconnected-(U2-PF1-Pad40) -> ROW3
- U2 pad 41: unconnected-(U2-PF0-Pad41) -> ROW4
Routing:
- net ROW4: track 209.6 -> 464.3 mm, vias 0 -> 1
- net ROW3: track 209.5 -> 443.9 mm, vias 0 -> 1
- net COL11: track 0.00 -> 230.8 mm
- net ROW2: track 209.6 -> 423.4 mm, vias 0 -> 1
- net COL10: track 0.00 -> 212.9 mm
- net COL9: track 0.00 -> 194.5 mm
- net ROW1: track 209.5 -> 403.1 mm, vias 0 -> 1
- net COL8: track 0.00 -> 175.8 mm
- net ROW0: track 209.6 -> 383.3 mm, vias 0 -> 1
- net COL7: track 0.00 -> 158.2 mm
- net COL0: track 0.00 -> 150.1 mm
- net COL6: track 0.00 -> 140.4 mm
- net COL1: track 0.00 -> 130.6 mm
- net COL5: track 0.00 -> 122.5 mm
- net GND: track 0.00 -> 120.2 mm, vias 0 -> 1
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Other:
- board outline added: 230.5 x 131 mm

Commit message: Daughter board
Put MCU and USB-C (+assoc. bits) on a daughter board to reduce overall footprint of pcb
Parts:
- added J2: Conn_01x17_Socket, Connector_PinHeader_1.00mm:PinHeader_1x17_P1.00mm_Horizontal, F.Cu at (122.0, 41.8)
- added J3: Conn_01x17_Socket, Connector_PinHeader_1.00mm:PinHeader_1x17_P1.00mm_Horizontal, F.Cu at (142.2, 4.60)
- moved C1 44.6 mm to (128.4, -20.2)
- moved C2 44.6 mm to (141.8, -5.77)
- moved C3 44.6 mm to (128.6, -0.77)
- moved C4 44.6 mm to (124.8, -18.0)
- moved C5 44.6 mm to (137.8, -19.0)
- moved C6 44.6 mm to (121.0, -6.77)
- moved C7 44.6 mm to (121.0, -13.3)
- moved R1 44.6 mm to (139.2, -0.02)
- moved R4 44.6 mm to (124.8, -21.3)
- moved SW1 44.6 mm to (135.6, -27.8)
- moved U2 44.6 mm to (132.8, -9.80)
- moved Y1 44.6 mm to (121.0, -10.0)
- moved R3 30.6 mm to (158.5, -4.19), turned to 90 degrees
- moved R2 29.5 mm to (156.3, -4.24), turned to 90 degrees
- moved R5 22.3 mm to (150.2, 0.61), turned to -90 degrees
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Connections:
- D1 pad 1: ROW0 -> ROW0.2
- D10 pad 1: ROW4 -> ROW4.2
- D11 pad 1: ROW0 -> ROW0.2
- D12 pad 1: ROW1 -> ROW1.2
- D13 pad 1: ROW2 -> ROW2.2
- D14 pad 1: ROW3 -> ROW3.2
- D15 pad 1: ROW4 -> ROW4.2
- D16 pad 1: ROW0 -> ROW0.2
- D17 pad 1: ROW1 -> ROW1.2
- D18 pad 1: ROW2 -> ROW2.2
- D19 pad 1: ROW3 -> ROW3.2
- D2 pad 1: ROW0 -> ROW0.2
- D20 pad 1: ROW4 -> ROW4.2
- D21 pad 1: ROW0 -> ROW0.2
- D22 pad 1: ROW1 -> ROW1.2
- D23 pad 1: ROW2 -> ROW2.2
- D24 pad 1: ROW3 -> ROW3.2
- D25 pad 1: ROW4 -> ROW4.2
- D26 pad 1: ROW0 -> ROW0.2
- D27 pad 1: ROW1 -> ROW1.2
- D28 pad 1: ROW2 -> ROW2.2
- D29 pad 1: ROW3 -> ROW3.2
- D3 pad 1: ROW1 -> ROW1.2
- D30 pad 1: ROW4 -> ROW4.2
- D31 pad 1: ROW0 -> ROW0.2
- D32 pad 1: ROW1 -> ROW1.2
- D33 pad 1: ROW2 -> ROW2.2
- D34 pad 1: ROW3 -> ROW3.2
- D35 pad 1: ROW4 -> ROW4.2
- D36 pad 1: ROW0 -> ROW0.2
- D37 pad 1: ROW1 -> ROW1.2
- D38 pad 1: ROW2 -> ROW2.2
- D39 pad 1: ROW3 -> ROW3.2
- D4 pad 1: ROW1 -> ROW1.2
- D40 pad 1: ROW4 -> ROW4.2
- D41 pad 1: ROW0 -> ROW0.2
- D42 pad 1: ROW1 -> ROW1.2
- D43 pad 1: ROW2 -> ROW2.2
- D44 pad 1: ROW3 -> ROW3.2
- D45 pad 1: ROW4 -> ROW4.2
- D46 pad 1: ROW0 -> ROW0.2
- D47 pad 1: ROW1 -> ROW1.2
- D48 pad 1: ROW2 -> ROW2.2
- D49 pad 1: ROW3 -> ROW3.2
- D5 pad 1: ROW2 -> ROW2.2
- D50 pad 1: ROW4 -> ROW4.2
- D51 pad 1: ROW0 -> ROW0.2
- D52 pad 1: ROW1 -> ROW1.2
- D53 pad 1: ROW2 -> ROW2.2
- D54 pad 1: ROW3 -> ROW3.2
- D55 pad 1: ROW4 -> ROW4.2
- D56 pad 1: ROW0 -> ROW0.2
- D57 pad 1: ROW1 -> ROW1.2
- D58 pad 1: ROW2 -> ROW2.2
- D59 pad 1: ROW3 -> ROW3.2
- D6 pad 1: ROW2 -> ROW2.2
- D60 pad 1: ROW4 -> ROW4.2
- D7 pad 1: ROW3 -> ROW3.2
- D8 pad 1: ROW3 -> ROW3.2
- D9 pad 1: ROW4 -> ROW4.2
- MX1 pad 1: COL0 -> COL0.2
- MX10 pad 1: COL1 -> COL1.2
- MX11 pad 1: COL2 -> COL2.2
- MX12 pad 1: COL2 -> COL2.2
- MX13 pad 1: COL2 -> COL2.2
- MX14 pad 1: COL2 -> COL2.2
- MX15 pad 1: COL2 -> COL2.2
- MX16 pad 1: COL3 -> COL3.2
- MX17 pad 1: COL3 -> COL3.2
- MX18 pad 1: COL3 -> COL3.2
- MX19 pad 1: COL3 -> COL3.2
- MX2 pad 1: COL1 -> COL1.2
- MX20 pad 1: COL3 -> COL3.2
- MX21 pad 1: COL4 -> COL4.2
- MX22 pad 1: COL4 -> COL4.2
- MX23 pad 1: COL4 -> COL4.2
- MX24 pad 1: COL4 -> COL4.2
- MX25 pad 1: COL4 -> COL4.2
- MX26 pad 1: COL5 -> COL5.2
- MX27 pad 1: COL5 -> COL5.2
- MX28 pad 1: COL5 -> COL5.2
- MX29 pad 1: COL5 -> COL5.2
- MX3 pad 1: COL0 -> COL0.2
- MX30 pad 1: COL5 -> COL5.2
- MX31 pad 1: COL6 -> COL6.2
- MX32 pad 1: COL6 -> COL6.2
- MX33 pad 1: COL6 -> COL6.2
- MX34 pad 1: COL6 -> COL6.2
- MX35 pad 1: COL6 -> COL6.2
- MX36 pad 1: COL7 -> COL7.2
- MX37 pad 1: COL7 -> COL7.2
- MX38 pad 1: COL7 -> COL7.2
- MX39 pad 1: COL7 -> COL7.2
- MX4 pad 1: COL1 -> COL1.2
- MX40 pad 1: COL7 -> COL7.2
- MX41 pad 1: COL8 -> COL8.2
- MX42 pad 1: COL8 -> COL8.2
- MX43 pad 1: COL8 -> COL8.2
- MX44 pad 1: COL8 -> COL8.2
- MX45 pad 1: COL8 -> COL8.2
- MX46 pad 1: COL9 -> COL9.2
- MX47 pad 1: COL9 -> COL9.2
- MX48 pad 1: COL9 -> COL9.2
- MX49 pad 1: COL9 -> COL9.2
- MX5 pad 1: COL0 -> COL0.2
- MX50 pad 1: COL9 -> COL9.2
- MX51 pad 1: COL10 -> COL10.2
- MX52 pad 1: COL10 -> COL10.2
- MX53 pad 1: COL10 -> COL10.2
- MX54 pad 1: COL10 -> COL10.2
- MX55 pad 1: COL10 -> COL10.2
- MX56 pad 1: COL11 -> COL11.2
- MX57 pad 1: COL11 -> COL11.2
- MX58 pad 1: COL11 -> COL11.2
- MX59 pad 1: COL11 -> COL11.2
- MX6 pad 1: COL1 -> COL1.2
- MX60 pad 1: COL11 -> COL11.2
- MX7 pad 1: COL0 -> COL0.2
- MX8 pad 1: COL1 -> COL1.2
- MX9 pad 1: COL0 -> COL0.2
- U2 pad 19: COL0 -> COL0.1
- U2 pad 20: COL1 -> COL1.1
- U2 pad 21: COL2 -> COL2.1
- U2 pad 22: COL3 -> COL3.1
- U2 pad 25: COL4 -> COL4.1
- U2 pad 26: COL5 -> COL5.1
- U2 pad 27: COL6 -> COL6.1
- U2 pad 28: COL7 -> COL7.1
- U2 pad 29: COL8 -> COL8.1
- U2 pad 30: COL9 -> COL9.1
- U2 pad 31: COL10 -> COL10.1
- U2 pad 32: COL11 -> COL11.1
- U2 pad 37: ROW0 -> ROW0.1
- U2 pad 38: ROW1 -> ROW1.1
- U2 pad 39: ROW2 -> ROW2.1
- U2 pad 40: ROW3 -> ROW3.1
- U2 pad 41: ROW4 -> ROW4.1
Routing:
- net ROW4: track 464.3 -> 0.00 mm, vias 1 -> 0
- net ROW4.2: track 0.00 -> 459.1 mm
- net ROW3: track 443.9 -> 0.00 mm, vias 1 -> 0
- net ROW3.2: track 0.00 -> 440.2 mm
- net ROW2: track 423.4 -> 0.00 mm, vias 1 -> 0
- net ROW2.2: track 0.00 -> 421.3 mm
- net ROW1: track 403.1 -> 0.00 mm, vias 1 -> 0
- net ROW1.2: track 0.00 -> 402.7 mm
- net ROW0.2: track 0.00 -> 384.6 mm
- net ROW0: track 383.3 -> 0.00 mm, vias 1 -> 0
- net COL11: track 230.8 -> 0.00 mm
- net COL11.2: track 0.00 -> 229.4 mm
- net COL10: track 212.9 -> 0.00 mm
- net COL10.2: track 0.00 -> 212.3 mm
- net COL9: track 194.5 -> 0.00 mm
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Other:
- board size 230.5 x 131 mm -> 237.2 x 177.3 mm

Commit message: lil bit of refining
Routing:
- net +5V: track 75.0 -> 106.2 mm
- net GND: track 83.9 -> 113.3 mm
